Commit message: inital simulation changes

File: description/lidar.xacro (robot description, xacro)
@@ -4,10 +4,10 @@
         <parent link="chassis"/>
         <child link="laser_frame"/>
-        <origin xyz="0.1 0 0.175" rpy="0 0 0"/>
+        <origin xyz="0.25 0 0.15" rpy="0 0 0"/>
     </joint>
     <link name="laser_frame">
         <visual>
             <geometry>
-                <cylinder radius="0.05" length="0.04"/>
+                <box size="0.08 0.08 0.04"/>
             </geometry>
             <material name="red"/>
@@ -15,10 +15,10 @@
         <collision>
             <geometry>
-                <cylinder radius="0.05" length="0.04"/>
+                <box size="0.08 0.08 0.04"/>
             </geometry>
         </collision>
-        <xacro:inertial_cylinder mass="0.1" length="0.04" radius="0.05">
+        <xacro:inertial_box mass="0.1" x="0.08" y="0.08" z="0.04">
             <origin xyz="0 0 0" rpy="0 0 0"/>
-        </xacro:inertial_cylinder>
+        </xacro:inertial_box>
     </link>
     <gazebo reference="laser_frame">
@@ -32,11 +32,11 @@
                     <horizontal>
                         <samples>360</samples>
-                        <min_angle>-3.14</min_angle>
-                        <max_angle>3.14</max_angle>
+                        <min_angle>-0.3927</min_angle>
+                        <max_angle>0.3927</max_angle>
                     </horizontal>
                 </scan>
                 <range>
                     <min>0.3</min>
-                    <max>12</max>
+                    <max>2</max>
                 </range>
             </ray>

File: description/robot.urdf.xacro (robot description, xacro)
@@ -3,4 +3,3 @@
     <xacro:include filename="robot_core.xacro" />
     <xacro:include filename="gazebo_control.xacro"/>
-    <xacro:include filename="lidar.xacro"/>
 </robot>

File: description/robot_core.xacro (robot description, xacro)
@@ -47,5 +47,5 @@
             </geometry>
         </collision>
-        <xacro:inertial_box mass="0.5" x ="0.5" y = "0.3" z = "0.15">
+        <xacro:inertial_box mass="0.5" x="0.3" y="0.3" z="0.1">
             <origin xyz="0.15 0.0 0.075" rpy="0.0 0.0 0.0"/>
         </xacro:inertial_box>
@@ -106,4 +106,31 @@
         <material>Gazebo/Blue</material>
     </gazebo>
+    <!--FRONT BOX LINK-->
+    <joint name="front_box_joint" type="fixed">
+        <parent link="chassis"/>
+        <child link="front_box"/>
+        <origin xyz="0.24 0.0 0.175"/>
+    </joint>
+    <link name="front_box">
+        <visual>
+            <origin xyz="0.0 0.0 0.0"/>
+            <geometry>
+                <box size="0.08 0.15 0.08"/>
+            </geometry>
+            <material name="red" />
+        </visual>
+        <collision>
+            <origin xyz="0.0 0.0 0.0"/>
+            <geometry>
+                <box size="0.08 0.15 0.08"/>
+            </geometry>
+        </collision>
+        <xacro:inertial_box mass="0.2" x="0.08" y="0.15" z="0.08">
+            <origin xyz="0.0 0.0 0.0" rpy="0.0 0.0 0.0"/>
+        </xacro:inertial_box>
+    </link>
+    <gazebo reference="front_box">
+        <material>Gazebo/Red</material>
+    </gazebo>
     <!--CASTER WHEEL LINK -->
     <joint name="caster_wheel_joint" type="fixed">
